File: aeropod2/aeropod2.kicad_pcb (KiCad board)
At the start: 4 copper layers, 41 x 90.2 mm, 67 parts, among them J1 USB_C_Receptacle_USB2.0_14P, J2 Conn_01x18, J4 AudioJack3_Ground, J5 Micro_SD_Card, J6 Conn_01x07, SW1 SW_Push_SPDT, SW2 SW_Push_SPDT, U1 TP4056-42-ESOP8, U2 AMS1117-3.3, U3 ESP32-WROOM-32, U4 MPR121QR2, U5 PCM5102A, U6 CP2102N-Axx-xQFN20, U7 MT3608

Commit message: Add fabrication outputs, printable case, and assembly guide
- Gerbers + drill files for both boards (aeropod2/gerbers, clickwheel/gerbers)
- BOM, pick-and-place positions, and JLC-ready zips in each production/ folder
- case/Aeropod_Case.step + .stl (both shells on one printable plate)
- ASSEMBLY.md with the step-by-step assembly plan; README fabrication section
Other:
- board text added: "aeropod"
- board text added: "evy 2026"
Changed lines of the file:
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@@
 			(plot_on_all_layers_selection 0x00000000_00000000_00000000_00000000)
 			(disableapertmacros no)
-			(usegerberextensions no)
+			(usegerberextensions yes)
 			(usegerberattributes yes)
 			(usegerberadvancedattributes yes)
@@
 			(outputformat 1)
 			(mirror no)
-			(drillshape 1)
+			(drillshape 0)
 			(scaleselection 1)
-			(outputdirectory "")
+			(outputdirectory "gerbers/")
 		)
 	)
@@
 			)
 		)
+		(property "LCSC Part #" ""
+			(at 0 0 0)
+			(unlocked yes)
+			(layer "F.Fab")
+			(hide yes)
+			(effects
+				(font
+					(size 1 1)
+					(thickness 0.15)
+				)
+			)
+		)
 		(property ki_fp_filters "ESP32?WROOM?32*")
 		(sheetname "/esp32/")
@@
 		(layer "Edge.Cuts")
 	)
+	(gr_text "evy 2026"
+		(at 113.0046 134.366 0)
+		(layer "F.SilkS")
+		(effects
+			(font
+				(size 1 1)
+				(thickness 0.1)
+			)
+			(justify left bottom)
+		)
+	)
+	(gr_text "aeropod"
+		(at 115.57 133.096 0)
+		(layer "F.SilkS")
+		(effects
+			(font
+				(size 1 1)
+				(thickness 0.1)
+			)
+			(justify left bottom)
+		)
+	)
 	(segment
