File: aeropod2/audio.kicad_sch (KiCad schematic)
At the start: 17 parts, among them J4 AudioJack3_Ground, U5 PCM5102A

Commit message: Restore the design files to the shipped revision
The earlier revert did not fully land: KiCad had the edited sheets open
and re-saved them over the restored files, so parts of the SD rewiring
and the B5 pin move were still present in audio, esp32 and storage.

All schematics, the board file and the firmware are now restored from
d6429d0 and verified by netlist comparison rather than by diffing text.
89 nets, electrically identical to the revision the gerbers and
production files were generated from. The SD socket is back to its
original wiring and the in-progress BQ24074 power work is reverted.

Also clears two stale KiCad lock files.
Other:
- note added: "In KiCad layout terms, what this actually means: On the PCB you draw a physical split in the ground plane under the PCM5102A, with the AGND copper pour on one side and the main DGND pour on the other. They connect at exactly one point - the star point, usually near the PCM5102A's GND pin. This stops ground return currents from the ESP32's SPI/I2S switching from flowing through the analog ground u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"
Changed lines of the file:
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@@
 	(generator_version "10.0")
 	(paper "A4")
+	(text "In KiCad layout terms, what this actually means:\nOn the PCB you draw a physical split in the ground plane under the PCM5102A, with the AGND copper pour on one side and the main DGND pour on the other. They connect at exactly one point - the star point, usually near the PCM5102A's GND pin. This stops ground return currents from the ESP32's SPI/I2S switching from flowing through the analog ground under the DAC's output pins, which is where they'd induce noise.\nThe AVDD decoupling caps (10 µF + 100 nF) should be placed on the AGND side of the split, as close to the AVDD pin as possible. If they're on the wrong side of the ferrite bead they're decoupling the wrong node.\nOne more thing the document glossed over - the charge pump caps (CAPP, CAMP, VNEG) also need to be on the AGND island, not the main ground plane. The charge pump generates a small negative voltage that lets the output swing below ground for a clean zero crossing, and that whole subcircuit needs to stay within the analog domain.\nFor a project like this the audible difference between doing this properly and just tying everything to a common ground is real - you'll hear it as a faint high-pitched whine or hash in quiet passages if the grounds aren't separated."
+		(exclude_from_sim no)
+		(at 150.622 154.432 0)
+		(effects
+			(font
+				(size 1.27 1.27)
+			)
+		)
+	)
 	(text "single star point to regular ground for agnd (pcb design step) look at claude chat"
 		(exclude_from_sim no)

Commit message: Rework the power options around battery life, not just correctness
The boost-then-LDO path on this board is the worst of the available
options for runtime: the MT3608 converts at about 88 percent and the
AMS1117 then burns the 4.8 V to 3.3 V difference as heat, so roughly 60
percent of the cell reaches the load. Repairing it is both the most
layout work and the least battery.

Documents four alternatives with rough energy numbers instead. The
default recommendation is now to delete the boost entirely and swap the
AMS1117 for an AP2114H-3.3, which is the same SOT-223 footprint and pin
order, needs no layout change, and still delivers more energy than the
repaired boost. Notes the AP2114HA variant, one letter different and
stocked alongside it, has a VIN/GND/VOUT pinout that would destroy the
board.

Also covers feeding the regulator straight from the cell for most of the
pack, a wired-in buck-boost module for the whole pack with no PCB work,
and a buck-boost IC as the proper fix for a respin.
Other:
- note removed: "In KiCad layout terms, what this actually means: On the PCB you draw a physical split in the ground plane under the PCM5102A, with the AGND copper pour on one side and the main DGND pour on the other. They connect at exactly one point - the star point, usually near the PCM5102A's GND pin. This stops ground return currents from the ESP32's SPI/I2S switching from flowing through the analog ground u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"
Changed lines of the file:
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@@
 	(generator_version "10.0")
 	(paper "A4")
-	(text "In KiCad layout terms, what this actually means:\nOn the PCB you draw a physical split in the ground plane under the PCM5102A, with the AGND copper pour on one side and the main DGND pour on the other. They connect at exactly one point - the star point, usually near the PCM5102A's GND pin. This stops ground return currents from the ESP32's SPI/I2S switching from flowing through the analog ground under the DAC's output pins, which is where they'd induce noise.\nThe AVDD decoupling caps (10 µF + 100 nF) should be placed on the AGND side of the split, as close to the AVDD pin as possible. If they're on the wrong side of the ferrite bead they're decoupling the wrong node.\nOne more thing the document glossed over - the charge pump caps (CAPP, CAMP, VNEG) also need to be on the AGND island, not the main ground plane. The charge pump generates a small negative voltage that lets the output swing below ground for a clean zero crossing, and that whole subcircuit needs to stay within the analog domain.\nFor a project like this the audible difference between doing this properly and just tying everything to a common ground is real - you'll hear it as a faint high-pitched whine or hash in quiet passages if the grounds aren't separated."
-		(exclude_from_sim no)
-		(at 150.622 154.432 0)
-		(effects
-			(font
-				(size 1.27 1.27)
-			)
-		)
-	)
 	(text "single star point to regular ground for agnd (pcb design step) look at claude chat"
 		(exclude_from_sim no)
