File: clickwheel/clickwheel.kicad_pcb (KiCad board)
At the start: 2 copper layers, 44.6 x 33.7 mm, 6 parts, among them J1 Conn_01x18, SW1 SW_Push, SW2 SW_Push, SW3 SW_Push, SW4 SW_Push, SW5 SW_Push

Commit message: Add fabrication outputs, printable case, and assembly guide
- Gerbers + drill files for both boards (aeropod2/gerbers, clickwheel/gerbers)
- BOM, pick-and-place positions, and JLC-ready zips in each production/ folder
- case/Aeropod_Case.step + .stl (both shells on one printable plate)
- ASSEMBLY.md with the step-by-step assembly plan; README fabrication section
Other:
- board text added: "clickwheel evy 26"
Changed lines of the file:
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@@
+			)
+		)
+		(property "LCSC Part #" ""
+			(at 0 0 0)
+			(unlocked yes)
+			(layer "B.Fab")
+			(hide yes)
+			(effects
+				(font
+					(size 1 1)
+					(thickness 0.15)
+				)
+				(justify mirror)
 			)
 		)
@@
 		(layer "Edge.Cuts")
 	)
+	(gr_text "clickwheel evy 26"
+		(at 117.4242 69.2658 0)
+		(layer "F.SilkS")
+		(effects
+			(font
+				(size 1 1)
+				(thickness 0.1)
+			)
+			(justify left bottom)
+		)
+	)
 	(segment
